File: ELECTRICAL/is-plant-okay/LoRA_RADIO.kicad_sch (KiCad schematic)
At the start: 0 parts

Commit message: feat: add lora
Parts:
- added U5: SX1276IMLTRT, is-plant-okay-foot:QFN65P600X600X100-29N, symbol is-plant-okay-lib:SX1276IMLTRT
Connections:
- new net GND: U5.15 (GND), U5.23 (GND__1), U5.26 (GND__2), U5.29 (GND__3)

Commit message: feat: add usb and esd protection device
Connections:
- net SCLK: now reaches U5.16 (SCK)
- net MISO: now reaches U5.17 (MISO)
- net MOSI: now reaches U5.18 (MOSI)
- net LORA_CS: now reaches U5.19 (NSS)
Changed lines of the file:
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@@
+	(wire
+		(pts
+			(xy 113.03 82.55) (xy 123.19 82.55)
+		)
+		(stroke
+			(width 0)
+			(type default)
+		)
+	)
 	(wire
 		(pts
 			(xy 172.72 118.11) (xy 172.72 120.65)
+		)
+		(stroke
+			(width 0)
+			(type default)
+		)
+	)
+	(wire
+		(pts
+			(xy 113.03 80.01) (xy 123.19 80.01)
 		)
 		(stroke
@@
 	(wire
 		(pts
+			(xy 113.03 74.93) (xy 123.19 74.93)
+		)
+		(stroke
+			(width 0)
+			(type default)
+		)
+	)
+	(wire
+		(pts
 			(xy 168.91 118.11) (xy 172.72 118.11)
 		)
@@
 		)
 	)
+	(wire
+		(pts
+			(xy 113.03 77.47) (xy 123.19 77.47)
+		)
+		(stroke
+			(width 0)
+			(type default)
+		)
+	)
+	(hierarchical_label "MISO"
+		(shape input)
+		(at 113.03 77.47 180)
+		(effects
+			(font
+				(size 1.27 1.27)
+			)
+			(justify right)
+		)
+	)
+	(hierarchical_label "SCLK"
+		(shape input)
+		(at 113.03 74.93 180)
+		(effects
+			(font
+				(size 1.27 1.27)
+			)
+			(justify right)
+		)
+	)
+	(hierarchical_label "LORA_CS"
+		(shape input)
+		(at 113.03 82.55 180)
+		(effects
+			(font
+				(size 1.27 1.27)
+			)
+			(justify right)
+		)
+	)
+	(hierarchical_label "MOSI"
+		(shape input)
+		(at 113.03 80.01 180)
+		(effects
+			(font
+				(size 1.27 1.27)
+			)
+			(justify right)
+		)
+	)
