File: ELECTRICAL/is-plant-okay/_autosave-LoRA_RADIO.kicad_sch (KiCad schematic)
At the start: 1 part, among them U9 Value

Commit message: feat: add ldo and power management IC
Changed lines of the file:
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@@
 	)
 	(hierarchical_label "3.3V"
-		(shape output)
+		(shape input)
 		(at 118.11 87.63 180)
 		(effects
