File: ELECTRICAL/is-plant-okay/USB_C_3-3V.kicad_sch (KiCad schematic)
At the start: 7 parts, among them J7 USB4085-GF-A_REVB, U6 USBLC6-2SC6

Commit message: feat: add remaining resistor, capacitor footprints
Parts:
- C11: value 4n7 1KV -> 4.7nF; footprint (none) -> is-plant-okay-foot:CAPC1005X55N; MANUFACTURER (none) -> Samsung Electro-Mechanics; MFG PART # (none) -> CL05B104KO5NNNC; PACKAGE (none) -> 0402; TYPE (none) -> SMD
Other:
- moved on the sheet: R3
Changed lines of the file:
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@@
-	)
-	(junction
-		(at 118.11 107.95)
-		(diameter 0)
-		(color 0 0 0 0)
 	)
 	(junction
@@
 	)
 	(junction
+		(at 114.3 107.95)
+		(diameter 0)
+		(color 0 0 0 0)
+	)
+	(junction
 		(at 121.92 105.41)
 		(diameter 0)
@@
 	(wire
 		(pts
-			(xy 118.11 107.95) (xy 118.11 111.76)
+			(xy 114.3 107.95) (xy 114.3 111.76)
 		)
 		(stroke
@@
 	(wire
 		(pts
-			(xy 99.06 107.95) (xy 118.11 107.95)
+			(xy 99.06 107.95) (xy 114.3 107.95)
 		)
 		(stroke
@@
 	(wire
 		(pts
-			(xy 118.11 119.38) (xy 118.11 127)
-		)
-		(stroke
-			(width 0)
-			(type default)
-		)
-	)
-	(wire
-		(pts
-			(xy 118.11 107.95) (xy 121.92 107.95)
+			(xy 114.3 119.38) (xy 114.3 127)
 		)
 		(stroke
@@
 		(pts
 			(xy 127 82.55) (xy 130.81 82.55)
+		)
+		(stroke
+			(width 0)
+			(type default)
+		)
+	)
+	(wire
+		(pts
+			(xy 114.3 107.95) (xy 121.92 107.95)
 		)
 		(stroke
@@
 			)
 		)
-		(property "Value" "4n7 1KV"
+		(property "Value" "4.7nF"
 			(at 102.87 116.8399 0)
 			(effects
@@
 			)
 		)
-		(property "Footprint" ""
+		(property "Footprint" "is-plant-okay-foot:CAPC1005X55N"
 			(at 100.0252 119.38 0)
 			(effects
@@
 			)
 		)
-		(property "Datasheet" "~"
+		(property "Datasheet" "https://jlcpcb.com/api/file/downloadByFileSystemAccessId/8579707269996871680"
 			(at 99.06 115.57 0)
 			(effects
@@
 			)
 		)
-		(property "Description" "Unpolarized capacitor"
+		(property "Description" "CAP CER 0.1UF 16V X7R 0402"
+			(at 99.06 115.57 0)
+			(effects
+				(font
+					(size 1.27 1.27)
+				)
+				(hide yes)
+			)
+		)
+		(property "MFG PART #" "CL05B104KO5NNNC"
+			(at 99.06 115.57 0)
+			(effects
+				(font
+					(size 1.27 1.27)
+				)
+				(hide yes)
+			)
+		)
+		(property "TYPE" "SMD"
+			(at 99.06 115.57 0)
+			(effects
+				(font
+					(size 1.27 1.27)
+				)
+				(hide yes)
+			)
+		)
+		(property "PACKAGE" "0402"
+			(at 99.06 115.57 0)
+			(effects
+				(font
+					(size 1.27 1.27)
+				)
+				(hide yes)
+			)
+		)
+		(property "MANUFACTURER" "Samsung Electro-Mechanics"
 			(at 99.06 115.57 0)
 			(effects
@@
 	(symbol
 		(lib_id "Device:R")
-		(at 118.11 115.57 0)
+		(at 114.3 115.57 0)
 		(unit 1)
 		(exclude_from_sim no)
@@
 		(fields_autoplaced yes)
 		(property "Reference" "R3"
-			(at 120.65 114.2999 0)
+			(at 116.84 114.2999 0)
 			(effects
 				(font
@@
 		)
 		(property "Value" "10K"
-			(at 120.65 116.8399 0)
+			(at 116.84 116.8399 0)
 			(effects
 				(font
@@
 		)
 		(property "Footprint" "is-plant-okay-foot:RC0805FR-7W10KL"
-			(at 116.332 115.57 90)
+			(at 112.522 115.57 90)
 			(effects
 				(font
@@
 		)
 		(property "Datasheet" "~https://www.yageogroup.com/content/datasheet/asset/file/PYU-RC_GROUP_51_ROHS_L"
-			(at 118.11 115.57 0)
+			(at 114.3 115.57 0)
 			(effects
 				(font
@@
 		)
 		(property "Description" "RES 10K OHM 1% 1/4W 0805"
-			(at 118.11 115.57 0)
+			(at 114.3 115.57 0)
 			(effects
 				(font
@@
 		)
 		(property "MFG PART #" "RC0805FR-7W10KL"
-			(at 118.11 115.57 0)
+			(at 114.3 115.57 0)
 			(effects
 				(font
@@
 		)
 		(property "TYPE" "SMD"
-			(at 118.11 115.57 0)
+			(at 114.3 115.57 0)
 			(effects
 				(font
@@
 		)
 		(property "PACKAGE" "0805"
-			(at 118.11 115.57 0)
+			(at 114.3 115.57 0)
 			(effects
 				(font
@@
 	(symbol
 		(lib_id "power:GND")
-		(at 118.11 127 0)
+		(at 114.3 127 0)
 		(unit 1)
 		(exclude_from_sim no)
@@
 		(fields_autoplaced yes)
 		(property "Reference" "#PWR033"
-			(at 118.11 133.35 0)
+			(at 114.3 133.35 0)
 			(effects
 				(font
@@
 		)
 		(property "Value" "GND"
-			(at 118.11 132.08 0)
+			(at 114.3 132.08 0)
 			(effects
 				(font
@@
 		)
 		(property "Footprint" ""
-			(at 118.11 127 0)
+			(at 114.3 127 0)
 			(effects
 				(font
@@
 		)
 		(property "Datasheet" ""
-			(at 118.11 127 0)
+			(at 114.3 127 0)
 			(effects
 				(font
@@
 		)
 		(property "Description" "Power symbol creates a global label with name \"GND\" , ground"
-			(at 118.11 127 0)
-			(effects
-				(font
+			(at 114.3 127 0)
+			(effects
+				(font
